File: DL_magnetometr/Digi_comp/Digi_comp.kicad_pcb (KiCad board)
At the start: 2 copper layers, 23 parts, among them J2 Conn_01x06_Male, U1 NUP2202, U5 AP7331-WG-7, U6 HC-06, U8 AP7331-WG-7, U9 ATmega328P-MU

Commit message: Layout continuation
Parts:
- removed the D1 at (42.3, 21.3)
- removed U5, U8: AP7331-WG-7, Package_TO_SOT_SMD:TSOT-23-5
- added C4: 1u, Capacitor_SMD:C_0805_2012Metric, F.Cu at (109.0, 38.0)
- added C5: 1u, Capacitor_SMD:C_0805_2012Metric, F.Cu at (71.2, 29.5)
- added F1: Fuse_Small, Fuse:Fuse_0805_2012Metric, F.Cu at (122.0, 42.0)
- added U3: AP7331-WG-7, Package_TO_SOT_SMD:TSOT-23-5, F.Cu at (115.0, 43.0)
- JP1: footprint Jumper:SolderJumper-3_P1.3mm_Bridged12_Pad1.0x1.5mm -> Jumper:SolderJumper-2_P1.3mm_Open_Pad1.0x1.5mm
- U1: value NUP2202 -> JST-PHR-2-Connector; footprint Package_TO_SOT_SMD:SOT-363_SC-70-6 -> Dokumenty:2AA-SM
- moved U2 112.6 mm to (132.0, 70.0), turned to 270 degrees
- moved U4 95.4 mm to (135.0, 48.0)
- moved J1 92.6 mm to (127.0, 37.0), turned to 90 degrees
- moved R7 71.8 mm to (122.0, 49.0)
- moved R8 63.5 mm to (116.0, 50.0), turned to 90 degrees
- moved U1 34.4 mm to (88.0, 44.0)
- renumbered C10 to C6, D2 to D1, J2 to J1, R3 to R1, R4 to R2, R14 to R3, R15 to R4, R16 to R5, R17 to R6, R18 to R7, R19 to R8, R20 to R9, U6 to U2, U9 to U4
Connections:
- C6 pad 1: 5V -> 3.3V
- J1 pad 2: 5V -> 3.3V
- U4 pad 18: 5V -> 3.3V
- U4 pad 4: 5V -> 3.3V
- U4 pad 6: 5V -> 3.3V

Commit message: Layout finished
Parts:
- removed U1: JST-PHR-2-Connector, Dokumenty:2AA-SM
- added BT1: Battery_Cell, Dokumenty:2AA-SM, F.Cu at (75.0, 65.0)
- added J2: Conn_01x01_Male, Connector_PinHeader_2.54mm:PinHeader_1x01_P2.54mm_Vertical, F.Cu at (103.5, 85.5)
- added J3: Conn_01x01_Male, Connector_PinHeader_2.54mm:PinHeader_1x01_P2.54mm_Vertical, F.Cu at (103.5, 81.5)
- added REF**: MountingHole_2.2mm_M2, MountingHole:MountingHole_2.2mm_M2, F.Cu at (112.0, 85.0)
- added REF**: MountingHole_2.2mm_M2, MountingHole:MountingHole_2.2mm_M2, F.Cu at (68.0, 85.0)
- added REF**: MountingHole_2.2mm_M2, MountingHole:MountingHole_2.2mm_M2, F.Cu at (112.0, 45.0)
- added REF**: MountingHole_2.2mm_M2, MountingHole:MountingHole_2.2mm_M2, F.Cu at (68.0, 45.0)
- moved D1 79.6 mm to (111.5, 79.5), turned to 270 degrees
- moved R4 78.8 mm to (107.5, 79.5), turned to 90 degrees
- moved R6 76.5 mm to (109.5, 79.5), turned to 90 degrees
- moved R3 75.2 mm to (99.5, 83.5), turned to 270 degrees
- moved JP1 72.1 mm to (95.0, 79.5), turned to 180 degrees
- moved R5 71.3 mm to (97.5, 83.5), turned to 90 degrees
- moved C6 70.7 mm to (110.5, 52.0), turned to 270 degrees
- moved R9 68.9 mm to (95.5, 83.5), turned to 270 degrees
- moved R1 62.8 mm to (97.5, 55.5), turned to 180 degrees
- moved R2 57.3 mm to (97.5, 57.5), turned to 180 degrees
- moved C2 54.3 mm to (88.0, 56.0), turned to 270 degrees
- moved C5 53.4 mm to (91.0, 79.0), turned to 90 degrees
- moved C3 51.9 mm to (95.0, 52.0), turned to 90 degrees
- moved S1 51.8 mm to (92.0, 55.0), turned to 180 degrees
- moved F1 49.6 mm to (89.0, 79.0), turned to 90 degrees
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Connections:
- R3 pad 2: (no net) -> Net-(J2-Pad1)
- R4 pad 1: (no net) -> Net-(J3-Pad1)
Routing:
- net 3.3V: track 0.00 -> 122.0 mm, vias 0 -> 3
- net GND: track 0.00 -> 39.5 mm, vias 0 -> 16
- net (no net): track 0.00 -> 35.8 mm
- net Net-(R4-Pad2): track 0.00 -> 19.4 mm, vias 0 -> 2
- net 3.6V: track 0.00 -> 18.6 mm
- net SCL: track 0.00 -> 15.1 mm, vias 0 -> 2
- net SDA: track 0.00 -> 14.8 mm
- net Net-(J1-Pad5): track 0.00 -> 13.2 mm, vias 0 -> 2
- net INT: track 0.00 -> 12.9 mm, vias 0 -> 2
- net Net-(C1-Pad2): track 0.00 -> 11.5 mm
- net Net-(J1-Pad1): track 0.00 -> 11.1 mm, vias 0 -> 2
- net Net-(JP1-Pad1): track 0.00 -> 10.8 mm
- net UART_RXD: track 0.00 -> 9.06 mm
- net UART_TXD: track 0.00 -> 8.87 mm
- net Net-(J1-Pad3): track 0.00 -> 6.72 mm
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- added copper zone on B.Cu, net GND
Other:
- board outline added: 50 x 46 mm
- net class Small added: clearance 0.2, trace_width 0.254, via_dia 0.8, via_drill 0.4

Commit message: Exit save
Routing:
- net 3.3V: track 122.0 -> 120.3 mm
- net INT: track 12.9 -> 13.7 mm
